Commit message: Connect robot visual geometry

File: ws/src/robotar_description/urdf/inc/base.xacro (robot description, xacro)
@@ -57,4 +57,13 @@
       <geometry><box size="0.075 ${BASE['wheel_width']+0.02} 0.036"/></geometry>
       <material name="lug_rubber"/>
+    </visual>
+  </xacro:macro>
+  <!-- Fixed visual axle connecting the chassis side to a wheel hub. The
+       physical wheel contact remains the wheel's own collision cylinder. -->
+  <xacro:macro name="wheel_axle" params="name px py">
+    <visual name="${name}">
+      <origin xyz="${px} ${math.copysign((BASE['wheel_track']/2.0 + CHASSIS['width']/2.0)/2.0, py)} ${BASE['wheel_radius'] - CHASSIS['center_height']}" rpy="${math.pi/2} 0 0"/>
+      <geometry><cylinder radius="0.045" length="${BASE['wheel_track']/2.0 - CHASSIS['width']/2.0 + 0.04}"/></geometry>
+      <material name="hub_steel"/>
     </visual>
   </xacro:macro>
@@ -161,4 +170,8 @@
       </collision>
     </link>
+    <xacro:wheel_axle name="fl_axle" px="${ BASE['wheelbase']/2.0}" py="${ BASE['wheel_track']/2.0}"/>
+    <xacro:wheel_axle name="rl_axle" px="${-BASE['wheelbase']/2.0}" py="${ BASE['wheel_track']/2.0}"/>
+    <xacro:wheel_axle name="fr_axle" px="${ BASE['wheelbase']/2.0}" py="${-BASE['wheel_track']/2.0}"/>
+    <xacro:wheel_axle name="rr_axle" px="${-BASE['wheelbase']/2.0}" py="${-BASE['wheel_track']/2.0}"/>
     <xacro:lugged_wheel link="fl_wheel_link" joint="${BASE['wheel_joints']['front_left']}"
                         px="${ BASE['wheelbase']/2.0}" py="${ BASE['wheel_track']/2.0}"/>

File: ws/src/robotar_description/urdf/inc/sensors.xacro (robot description, xacro)
@@ -20,5 +20,5 @@
     <link name="mast_link">
       <!-- Pole runs from the chassis deck up to the mast head. -->
-      <xacro:property name="deck_z" value="${CHASSIS['center_height'] + CHASSIS['height']/2.0}"/>
+      <xacro:property name="deck_z" value="${CHASSIS['height']/2.0}"/>
       <xacro:property name="pole_len" value="${MAST['xyz'][2] - deck_z}"/>
       <xacro:inertial_cylinder_z mass="4.0" radius="0.035" length="${pole_len}" oz="${-pole_len/2.0}"/>
@@ -26,4 +26,9 @@
         <origin xyz="0 0 ${-pole_len/2.0}" rpy="0 0 0"/>
         <geometry><cylinder radius="0.035" length="${pole_len}"/></geometry>
+        <material name="mast_steel"/>
+      </visual>
+      <visual name="neck">
+        <origin xyz="0 0 ${(MAST['camera_xyz'][2] - 0.03)/2.0}" rpy="0 0 0"/>
+        <geometry><cylinder radius="0.03" length="${MAST['camera_xyz'][2] - 0.03}"/></geometry>
         <material name="mast_steel"/>
       </visual>

File: ws/src/robotar_description/urdf/tools/comb.xacro (robot description, xacro)
@@ -77,4 +77,9 @@
                           sx="${COMB['size'][0]}" sy="${COMB['size'][1]}" sz="${COMB['size'][2]}"
                           oz="${0.02 + COMB['size'][2]/2.0}"/>
+      <visual name="flange_adapter">
+        <origin xyz="0 0 0" rpy="0 0 0"/>
+        <geometry><cylinder radius="${R['flange']['bolt_circle_diameter']/2.0 + 0.005}" length="0.04"/></geometry>
+        <material name="hub_steel"/>
+      </visual>
       <visual name="top_guard_plate">
         <origin xyz="0 0 ${COMB['size'][2]}" rpy="0 0 0"/>
