Commit message: Close arm and sensor visual gaps

File: ws/src/robotar_description/urdf/inc/arm.xacro (robot description, xacro)
@@ -14,5 +14,7 @@
 -->
 <robot xmlns:xacro="http://www.ros.org/wiki/xacro">
-  <!-- Box arm segment extending along +x from its parent joint. -->
+  <!-- Box arm segment extending along +x from its parent joint, with a
+       visual bearing cap covering the proximal joint seam. The cap is
+       visual-only so it does not change the validated contact behavior. -->
   <xacro:macro name="arm_segment" params="link length width height mass">
     <link name="${link}">
@@ -23,4 +25,9 @@
         <geometry><box size="${length} ${width} ${height}"/></geometry>
         <material name="arm_orange"/>
+      </visual>
+      <visual name="proximal_bearing">
+        <origin xyz="0 0 0" rpy="${math.pi/2} 0 0"/>
+        <geometry><cylinder radius="${height/2.0 + 0.01}" length="${width + 0.02}"/></geometry>
+        <material name="arm_dark"/>
       </visual>
       <collision name="${link}_collision">
@@ -52,13 +59,17 @@
     </joint>
     <link name="arm_base_link">
-      <xacro:inertial_cylinder_z mass="6.0" radius="0.11" length="0.16" oz="-0.05"/>
+      <xacro:property name="pedestal_bottom" value="${CHASSIS['height']/2.0 - ARM['mount_xyz'][2]}"/>
+      <xacro:property name="pedestal_top" value="0.08"/>
+      <xacro:property name="pedestal_length" value="${pedestal_top - pedestal_bottom}"/>
+      <xacro:property name="pedestal_center" value="${(pedestal_top + pedestal_bottom)/2.0}"/>
+      <xacro:inertial_cylinder_z mass="8.0" radius="0.11" length="${pedestal_length}" oz="${pedestal_center}"/>
       <visual name="pedestal">
-        <origin xyz="0 0 -0.05" rpy="0 0 0"/>
-        <geometry><cylinder radius="0.11" length="0.16"/></geometry>
+        <origin xyz="0 0 ${pedestal_center}" rpy="0 0 0"/>
+        <geometry><cylinder radius="0.11" length="${pedestal_length}"/></geometry>
         <material name="arm_dark"/>
       </visual>
       <collision name="arm_base_collision">
-        <origin xyz="0 0 -0.05" rpy="0 0 0"/>
-        <geometry><cylinder radius="0.11" length="0.16"/></geometry>
+        <origin xyz="0 0 ${pedestal_center}" rpy="0 0 0"/>
+        <geometry><cylinder radius="0.11" length="${pedestal_length}"/></geometry>
       </collision>
     </link>

File: ws/src/robotar_description/urdf/inc/sensors.xacro (robot description, xacro)
@@ -123,5 +123,14 @@
     </joint>
     <link name="${IMU['link']}">
+      <xacro:property name="imu_bracket_bottom" value="${CHASSIS['height']/2.0 - IMU['xyz'][2]}"/>
+      <xacro:property name="imu_bracket_top" value="-0.015"/>
+      <xacro:property name="imu_bracket_length" value="${imu_bracket_top - imu_bracket_bottom}"/>
+      <xacro:property name="imu_bracket_center" value="${(imu_bracket_top + imu_bracket_bottom)/2.0}"/>
       <xacro:inertial_box mass="0.1" sx="0.05" sy="0.05" sz="0.03"/>
+      <visual name="mounting_bracket">
+        <origin xyz="0 0 ${imu_bracket_center}" rpy="0 0 0"/>
+        <geometry><box size="0.08 0.08 ${imu_bracket_length}"/></geometry>
+        <material name="mast_steel"/>
+      </visual>
       <visual name="pod">
         <origin xyz="0 0 0" rpy="0 0 0"/>
@@ -129,4 +138,8 @@
         <material name="sensor_black"/>
       </visual>
+      <collision name="imu_bracket_collision">
+        <origin xyz="0 0 ${imu_bracket_center}" rpy="0 0 0"/>
+        <geometry><box size="0.08 0.08 ${imu_bracket_length}"/></geometry>
+      </collision>
       <collision name="imu_collision">
         <origin xyz="0 0 0" rpy="0 0 0"/>
