Commit message: Add branch clamp-shaker tool and shaker mission state machine
Enclosed padded-jaw clamp + counter-rotating eccentric rotors behind the
tool0 flange (comb kept as legacy demo). Compliant spring/damper target
branch, clamp-verification contact gate, 10-25 Hz sweep + 4 s shake
mission, miss-contact negative mode. APPROACH wrist-limit latching fixed
via widened wrist_pitch range, >= 0.15 rad pose margins and a slide
midpoint; end-to-end validation still in progress (see DEVELOPMENT_LOG).

File: ws/src/robotar_description/urdf/inc/ros2_control.xacro (robot description, xacro)
@@ -9,4 +9,7 @@
     gripper (mimic)   : state only; GazeboSimSystem follows the URDF
                         <mimic> element for gripper_right_joint
+    shaker rotors     : velocity command, position+velocity state
+    shaker clamp jaw  : position command, position+velocity state
+    shaker mimic jaw  : state only (mimic of the commanded jaw)
   The gz_ros2_control Gazebo plugin block is emitted only when a
   controllers_file path is supplied, so the description stays usable for
@@ -66,4 +69,25 @@
         </joint>
       </xacro:if>
+      <xacro:if value="${tool == 'shaker'}">
+        <joint name="${SHAKER['clamp']['commanded_joint']}">
+          <command_interface name="position"/>
+          <state_interface name="position"/>
+          <state_interface name="velocity"/>
+        </joint>
+        <joint name="${SHAKER['clamp']['mimic_joint']}">
+          <state_interface name="position"/>
+          <state_interface name="velocity"/>
+        </joint>
+        <joint name="${SHAKER['rotors']['joints'][0]}">
+          <command_interface name="velocity"/>
+          <state_interface name="position"/>
+          <state_interface name="velocity"/>
+        </joint>
+        <joint name="${SHAKER['rotors']['joints'][1]}">
+          <command_interface name="velocity"/>
+          <state_interface name="position"/>
+          <state_interface name="velocity"/>
+        </joint>
+      </xacro:if>
     </ros2_control>
     <xacro:if value="${controllers_file != ''}">
@@ -71,4 +95,7 @@
         <plugin filename="gz_ros2_control-system" name="gz_ros2_control::GazeboSimROS2ControlPlugin">
           <parameters>${controllers_file}</parameters>
+          <!-- Position-servo P gain from the physical.yaml SSOT (see the
+               control.position_proportional_gain comment there). -->
+          <position_proportional_gain>${CONTROL['position_proportional_gain']}</position_proportional_gain>
         </plugin>
       </gazebo>

File: ws/src/robotar_description/urdf/robotar.urdf.xacro (robot description, xacro)
@@ -7,6 +7,7 @@
   together; it contains no duplicated physical constants.
   Arguments:
-    tool             : 'comb' (default) or 'gripper' — launch-time tool
-                       interchangeability behind the common tool0 flange.
+    tool             : 'comb' (default), 'gripper' or 'shaker' — launch-time
+                       tool interchangeability behind the common tool0
+                       flange.
     physical_params  : path to the SSOT YAML (default: the package copy,
                        resolved relative to this file).
@@ -25,6 +26,6 @@
        tool selection (xacro properties are lazy; an element attribute is
        evaluated eagerly when this conditional body is emitted). -->
-  <xacro:unless value="${'$(arg tool)' == 'comb' or '$(arg tool)' == 'gripper'}">
-    <link name="unsupported_tool_${{'comb': 'comb', 'gripper': 'gripper'}['$(arg tool)']}"/>
+  <xacro:unless value="${'$(arg tool)' == 'comb' or '$(arg tool)' == 'gripper' or '$(arg tool)' == 'shaker'}">
+    <link name="unsupported_tool_${{'comb': 'comb', 'gripper': 'gripper', 'shaker': 'shaker'}['$(arg tool)']}"/>
   </xacro:unless>
   <!-- SSOT handles; every subsystem macro reads through these. -->
@@ -40,5 +41,7 @@
   <xacro:property name="COMB" value="${R['tools']['comb']}"/>
   <xacro:property name="GRIPPER" value="${R['tools']['gripper']}"/>
+  <xacro:property name="SHAKER" value="${R['tools']['shaker']}"/>
   <xacro:property name="SENSORS" value="${R['sensors']}"/>
+  <xacro:property name="CONTROL" value="${ROBOTAR_CFG['control']}"/>
   <xacro:property name="TOPICS" value="${ROBOTAR_CFG['topics']}"/>
   <!-- Global color palette; subsystem files reference these by name. -->
@@ -57,4 +60,8 @@
   <material name="rotor_dark"><color rgba="0.15 0.15 0.16 1.0"/></material>
   <material name="comb_guard"><color rgba="0.72 0.55 0.10 1.0"/></material>
+  <!-- Shaker: translucent teal enclosure so the counter-rotating eccentric
+       discs (bright yellow) stay readable inside the housing. -->
+  <material name="shaker_housing"><color rgba="0.10 0.45 0.50 0.40"/></material>
+  <material name="shaker_rotor"><color rgba="0.85 0.65 0.10 1.0"/></material>
   <!-- Relative include paths resolve against this file's directory. -->
   <xacro:include filename="inc/base.xacro"/>
@@ -64,4 +71,5 @@
   <xacro:include filename="tools/comb.xacro"/>
   <xacro:include filename="tools/gripper.xacro"/>
+  <xacro:include filename="tools/shaker.xacro"/>
   <!-- Root of the TF tree: ground projection of the chassis center. -->
   <link name="base_footprint"/>
@@ -80,4 +88,7 @@
     <xacro:robotar_gripper_tool/>
   </xacro:if>
+  <xacro:if value="${'$(arg tool)' == 'shaker'}">
+    <xacro:robotar_shaker_tool/>
+  </xacro:if>
   <xacro:robotar_ros2_control tool="$(arg tool)" controllers_file="$(arg controllers_file)"/>
 </robot>
